Commit message: Fixes

File: urdf/sick_lms1xx.urdf.xacro (robot description, xacro)
@@ -25,7 +25,6 @@
 SOFTWARE, EVEN IF ADVISED OF THE POSSIBILITY OF SUCH DAMAGE.
 -->
-<robot xmlns:xacro="http://www.ros.org/wiki/xacro">
-  <xacro:macro name="sick_lms1xx" params="frame:=laser topic:=scan sample_size:=720 update_rate:=50
-               min_angle:=-2.35619 max_angle:=2.35619 min_range:=0.1 max_range:=30.0 robot_namespace:=/" >
+<robot xmlns:xacro="http://ros.org/wiki/xacro">
+  <xacro:macro name="sick_lms1xx" params="frame:=laser topic:=scan sample_size:=720 update_rate:=50 min_range:=0.1 max_range:=30.0 robot_namespace:=/" >
     <link name="${frame}">
       <inertial>
@@ -61,6 +60,6 @@
               <samples>${sample_size}</samples>
               <resolution>1</resolution>
-              <min_angle>${min_angle}</min_angle>
-              <max_angle>${max_angle}</max_angle>
+              <min_angle>-2.35619</min_angle>
+              <max_angle>2.35619</max_angle>
             </horizontal>
           </scan>
